Commit message: 模型debug2中添加kinect

File: barrett_model/robots/debug2_wam_7dof_wam_bhand.urdf.xacro (robot description, xacro)
@@ -335,421 +335,7 @@
     </inertial>
   </link>
-  <joint name="wam/bhand/bhand_base_joint" type="fixed">
-    <parent link="wam/wrist_palm_link"/>
-    <child link="wam/bhand/bhand_palm_link"/>
-    <origin rpy="0 0 3.14159265359" xyz="0 0 0.06"/>
-  </joint>
-  <gazebo reference="wam/bhand/bhand_palm_link">
-    <mu1>0.8</mu1>
-    <mu2>0.8</mu2>
-  </gazebo>
-  <link name="wam/bhand/bhand_palm_link">
-    <inertial>
-      <origin xyz="-5.1098e-005 0.0050433 0.036671"/>
-      <mass value="0.50573"/>
-      <inertia ixx="3.8374e-005" ixy="-5.604e-008" ixz="-4.2034e-005" iyy="0.00022405" iyz="1.3283e-007" izz="0.00020045"/>
-    </inertial>
-    <visual>
-      <material name="WAMGrey">
-        <color rgba="0.9 0.9 0.9 0.0"/>
-      </material>
-      <geometry>
-        <mesh filename="package://barrett_model/models/sw_meshes/bhand/bhand_palm_fine.stl"/>
-      </geometry>
-    </visual>
-    <collision>
-      <geometry>
-        <mesh filename="package://barrett_model/models/sw_meshes/bhand/bhand_palm_link_convex_decomposition.dae"/>
-      </geometry>
-    </collision>
-  </link>
-  <joint name="wam/bhand/bhand_palm_surface_joint" type="fixed">
-    <parent link="wam/bhand/bhand_palm_link"/>
-    <child link="wam/bhand/bhand_palm_surface_link"/>
-    <origin rpy="0 0 0" xyz="0 0 0.08"/>
-    <limit effort="5" lower="0" upper="3.14159265359" velocity="5.0"/>
-    <dynamics damping="0.11" friction="0"/>
-  </joint>
-  <link name="wam/bhand/bhand_palm_surface_link">
-    <inertial>
-      <mass value="0.000001"/>
-      <inertia ixx="0.000001" ixy="0.0" ixz="0.0" iyy="0.000001" iyz="0.0" izz="0.000001"/>
-    </inertial>
-  </link>
-  <joint name="wam/bhand/bhand_grasp_joint" type="fixed">
-    <parent link="wam/bhand/bhand_palm_link"/>
-    <child link="wam/bhand/bhand_grasp_link"/>
-    <origin rpy="0 0 0" xyz="0 0 0.12"/>
-    <limit effort="5" lower="0" upper="3.14159265359" velocity="5.0"/>
-    <dynamics damping="0.11" friction="0"/>
-  </joint>
-  <link name="wam/bhand/bhand_grasp_link">
-    <inertial>
-      <mass value="0.000001"/>
-      <inertia ixx="0.000001" ixy="0.0" ixz="0.0" iyy="0.000001" iyz="0.0" izz="0.000001"/>
-    </inertial>
-  </link>
-  <joint name="wam/bhand/finger_1/prox_joint" type="revolute">
-    <parent link="wam/bhand/bhand_palm_link"/>
-    <child link="wam/bhand/finger_1/prox_link"/>
-    <origin rpy="0 0 -1.57079632679" xyz="-0.025 0.0 0.0415"/>
-    <axis xyz="0 0 -1"/>
-    <limit effort="5" lower="0" upper="3.14159265359" velocity="5.0"/>
-    <dynamics damping="0.11" friction="0"/>
-  </joint>
-  <gazebo reference="wam/bhand/finger_1/prox_joint">
-    <provideFeedback>true</provideFeedback>
-    <implicitSpringDamper>true</implicitSpringDamper>
-    <!--<kp>0.0</kp>[> CFM <]-->
-    <!--<kd>0.0</kd>[> ERP <]-->
-    <!--<cfmDamping>true</cfmDamping>-->
-    <!--<dynamics damping="5.5" friction="1"/>-->
-  </gazebo>
-  <gazebo reference="wam/bhand/finger_1/prox_link">
-    <mu1>0.8</mu1>
-    <mu2>0.8</mu2>
-  </gazebo>
-  <link name="wam/bhand/finger_1/prox_link">
-    <inertial>
-      <origin xyz="0.023133 0.00078642 0.00052792"/>
-      <mass value="0.14109"/>
-      <inertia ixx="4.872e-006" ixy="1.7103e-006" ixz="3.4041e-008" iyy="7.6588e-005" iyz="2.3133e-008" izz="7.7733e-005"/>
-    </inertial>
-    <visual>
-      <material name="WAMGrey">
-        <color rgba="0.9 0.9 0.9 0.0"/>
-      </material>
-      <geometry>
-        <mesh filename="package://barrett_model/models/sw_meshes/bhand/bhand_finger_prox_link_fine.stl"/>
-      </geometry>
-    </visual>
-    <collision>
-      <geometry>
-        <mesh filename="package://barrett_model/models/sw_meshes/bhand/bhand_finger_prox_link_convex_decomposition.dae"/>
-      </geometry>
-    </collision>
-  </link>
-  <joint name="wam/bhand/finger_1/med_joint" type="revolute">
-    <parent link="wam/bhand/finger_1/prox_link"/>
-    <child link="wam/bhand/finger_1/med_link"/>
-    <origin rpy="1.57079632679 0 0" xyz="0.05 0.0 0.03390"/>
-    <axis xyz="0 0 1"/>
-    <limit effort="5" lower="0" upper="2.44346095279" velocity="5.00"/>
-    <dynamics damping="0.11" friction="0"/>
-  </joint>
-  <gazebo reference="wam/bhand/finger_1/med_joint">
-    <provideFeedback>true</provideFeedback>
-    <implicitSpringDamper>true</implicitSpringDamper>
-    <!--<kp>0.0</kp>[> CFM <]-->
-    <!--<kd>0.0</kd>[> ERP <]-->
-    <!--<cfmDamping>true</cfmDamping>-->
-    <!--<dynamics damping="5.5" friction="1"/>-->
-  </gazebo>
-  <gazebo reference="wam/bhand/finger_1/med_link">
-    <mu1>0.8</mu1>
-    <mu2>0.8</mu2>
-  </gazebo>
-  <link name="wam/bhand/finger_1/med_link">
-    <inertial>
-      <origin xyz="0.023133 0.00078642 0.00052792"/>
-      <mass value="0.062139"/>
-      <inertia ixx="4.872e-006" ixy="1.7103e-006" ixz="3.4041e-008" iyy="7.6588e-005" iyz="2.3133e-008" izz="7.7733e-005"/>
-    </inertial>
-    <visual>
-      <material name="WAMGrey">
-        <color rgba="0.9 0.9 0.9 0.0"/>
-      </material>
-      <geometry>
-        <mesh filename="package://barrett_model/models/sw_meshes/bhand/bhand_finger_med_link_fine.stl"/>
-      </geometry>
-    </visual>
-    <collision>
-      <geometry>
-        <mesh filename="package://barrett_model/models/sw_meshes/bhand/bhand_finger_med_link_convex.dae"/>
-      </geometry>
-    </collision>
-  </link>
-  <joint name="wam/bhand/finger_1/dist_joint" type="revolute">
-    <parent link="wam/bhand/finger_1/med_link"/>
-    <child link="wam/bhand/finger_1/dist_link"/>
-    <origin rpy="0 0 0.785398163397" xyz="0.06994 0.003 0.0"/>
-    <axis xyz="0 0 1"/>
-    <limit effort="5" lower="0" upper="0.837758040957" velocity="5.00"/>
-    <dynamics damping="0.11" friction="0"/>
-  </joint>
-  <gazebo reference="wam/bhand/finger_1/dist_joint">
-    <provideFeedback>true</provideFeedback>
-    <implicitSpringDamper>true</implicitSpringDamper>
-    <!--<kp>0.0</kp>[> CFM <]-->
-    <!--<kd>0.0</kd>[> ERP <]-->
-    <!--<cfmDamping>true</cfmDamping>-->
-    <!--<dynamics damping="5.5" friction="1"/>-->
-  </gazebo>
-  <gazebo reference="wam/bhand/finger_1/dist_link">
-    <mu1>0.8</mu1>
-    <mu2>0.8</mu2>
-    <selfCollide>true</selfCollide>
-  </gazebo>
-  <link name="wam/bhand/finger_1/dist_link">
-    <inertial>
-      <origin rpy="0 0 0" xyz="0.022825 0.0010491 0.0004203"/>
-      <mass value="0.041377"/>
-      <inertia ixx="3.1582e-006" ixy="1.4308e-006" ixz="1.0106e-007" iyy="3.8376e-005" iyz="0" izz="3.7275e-005"/>
-    </inertial>
-    <visual>
-      <origin rpy="0 0 -0.785398163397"/>
-      <material name="WAMGrey">
-        <color rgba="0.9 0.9 0.9 0.0"/>
-      </material>
-      <geometry>
-        <mesh filename="package://barrett_model/models/sw_meshes/bhand/bhand_finger_dist_link_fine.stl"/>
-      </geometry>
-    </visual>
-    <collision>
-      <origin rpy="0 0 -0.785398163397"/>
-      <geometry>
-        <mesh filename="package://barrett_model/models/sw_meshes/bhand/bhand_finger_dist_link_convex.dae"/>
-      </geometry>
-    </collision>
-  </link>
-  <joint name="wam/bhand/finger_1/tip_joint" type="fixed">
-    <parent link="wam/bhand/finger_1/dist_link"/>
-    <child link="wam/bhand/finger_1/tip_link"/>
-    <origin rpy="0 0 0" xyz="0.05 0.0 0.0"/>
-  </joint>
-  <link name="wam/bhand/finger_1/tip_link">
-    <inertial>
-      <mass value="1E-6"/>
-      <inertia ixx="1E-6" ixy="0" ixz="0" iyy="1E-6" iyz="0" izz="1E-6"/>
-    </inertial>
-  </link>
-  <joint name="wam/bhand/finger_2/prox_joint" type="revolute">
-    <parent link="wam/bhand/bhand_palm_link"/>
-    <child link="wam/bhand/finger_2/prox_link"/>
-    <origin rpy="0 0 -1.57079632679" xyz="0.025 0.0 0.0415"/>
-    <axis xyz="0 0 1"/>
-    <limit effort="5" lower="0" upper="3.14159265359" velocity="5.0"/>
-    <dynamics damping="0.11" friction="0"/>
-  </joint>
-  <gazebo reference="wam/bhand/finger_2/prox_joint">
-    <provideFeedback>true</provideFeedback>
-    <implicitSpringDamper>true</implicitSpringDamper>
-    <!--<kp>0.0</kp>[> CFM <]-->
-    <!--<kd>0.0</kd>[> ERP <]-->
-    <!--<cfmDamping>true</cfmDamping>-->
-    <!--<dynamics damping="5.5" friction="1"/>-->
-  </gazebo>
-  <gazebo reference="wam/bhand/finger_2/prox_link">
-    <mu1>0.8</mu1>
-    <mu2>0.8</mu2>
-  </gazebo>
-  <link name="wam/bhand/finger_2/prox_link">
-    <inertial>
-      <origin xyz="0.023133 0.00078642 0.00052792"/>
-      <mass value="0.14109"/>
-      <inertia ixx="4.872e-006" ixy="1.7103e-006" ixz="3.4041e-008" iyy="7.6588e-005" iyz="2.3133e-008" izz="7.7733e-005"/>
-    </inertial>
-    <visual>
-      <material name="WAMGrey">
-        <color rgba="0.9 0.9 0.9 0.0"/>
-      </material>
-      <geometry>
-        <mesh filename="package://barrett_model/models/sw_meshes/bhand/bhand_finger_prox_link_fine.stl"/>
-      </geometry>
-    </visual>
-    <collision>
-      <geometry>
-        <mesh filename="package://barrett_model/models/sw_meshes/bhand/bhand_finger_prox_link_convex_decomposition.dae"/>
-      </geometry>
-    </collision>
-  </link>
-  <joint name="wam/bhand/finger_2/med_joint" type="revolute">
-    <parent link="wam/bhand/finger_2/prox_link"/>
-    <child link="wam/bhand/finger_2/med_link"/>
-    <origin rpy="1.57079632679 0 0" xyz="0.05 0.0 0.03390"/>
-    <axis xyz="0 0 1"/>
-    <limit effort="5" lower="0" upper="2.44346095279" velocity="5.00"/>
-    <dynamics damping="0.11" friction="0"/>
-  </joint>
-  <gazebo reference="wam/bhand/finger_2/med_joint">
-    <provideFeedback>true</provideFeedback>
-    <implicitSpringDamper>true</implicitSpringDamper>
-    <!--<kp>0.0</kp>[> CFM <]-->
-    <!--<kd>0.0</kd>[> ERP <]-->
-    <!--<cfmDamping>true</cfmDamping>-->
-    <!--<dynamics damping="5.5" friction="1"/>-->
-  </gazebo>
-  <gazebo reference="wam/bhand/finger_2/med_link">
-    <mu1>0.8</mu1>
-    <mu2>0.8</mu2>
-  </gazebo>
-  <link name="wam/bhand/finger_2/med_link">
-    <inertial>
-      <origin xyz="0.023133 0.00078642 0.00052792"/>
-      <mass value="0.062139"/>
-      <inertia ixx="4.872e-006" ixy="1.7103e-006" ixz="3.4041e-008" iyy="7.6588e-005" iyz="2.3133e-008" izz="7.7733e-005"/>
-    </inertial>
-    <visual>
-      <material name="WAMGrey">
-        <color rgba="0.9 0.9 0.9 0.0"/>
-      </material>
-      <geometry>
-        <mesh filename="package://barrett_model/models/sw_meshes/bhand/bhand_finger_med_link_fine.stl"/>
-      </geometry>
-    </visual>
-    <collision>
-      <geometry>
-        <mesh filename="package://barrett_model/models/sw_meshes/bhand/bhand_finger_med_link_convex.dae"/>
-      </geometry>
-    </collision>
-  </link>
-  <joint name="wam/bhand/finger_2/dist_joint" type="revolute">
-    <parent link="wam/bhand/finger_2/med_link"/>
-    <child link="wam/bhand/finger_2/dist_link"/>
-    <origin rpy="0 0 0.785398163397" xyz="0.06994 0.003 0.0"/>
-    <axis xyz="0 0 1"/>
-    <limit effort="5" lower="0" upper="0.837758040957" velocity="5.00"/>
-    <dynamics damping="0.11" friction="0"/>
-  </joint>
-  <gazebo reference="wam/bhand/finger_2/dist_joint">
-    <provideFeedback>true</provideFeedback>
-    <implicitSpringDamper>true</implicitSpringDamper>
-    <!--<kp>0.0</kp>[> CFM <]-->
-    <!--<kd>0.0</kd>[> ERP <]-->
-    <!--<cfmDamping>true</cfmDamping>-->
-    <!--<dynamics damping="5.5" friction="1"/>-->
-  </gazebo>
-  <gazebo reference="wam/bhand/finger_2/dist_link">
-    <mu1>0.8</mu1>
-    <mu2>0.8</mu2>
-    <selfCollide>true</selfCollide>
-  </gazebo>
-  <link name="wam/bhand/finger_2/dist_link">
-    <inertial>
-      <origin rpy="0 0 0" xyz="0.022825 0.0010491 0.0004203"/>
-      <mass value="0.041377"/>
-      <inertia ixx="3.1582e-006" ixy="1.4308e-006" ixz="1.0106e-007" iyy="3.8376e-005" iyz="0" izz="3.7275e-005"/>
-    </inertial>
-    <visual>
-      <origin rpy="0 0 -0.785398163397"/>
-      <material name="WAMGrey">
-        <color rgba="0.9 0.9 0.9 0.0"/>
-      </material>
-      <geometry>
-        <mesh filename="package://barrett_model/models/sw_meshes/bhand/bhand_finger_dist_link_fine.stl"/>
-      </geometry>
-    </visual>
-    <collision>
-      <origin rpy="0 0 -0.785398163397"/>
-      <geometry>
-        <mesh filename="package://barrett_model/models/sw_meshes/bhand/bhand_finger_dist_link_convex.dae"/>
-      </geometry>
-    </collision>
-  </link>
-  <joint name="wam/bhand/finger_2/tip_joint" type="fixed">
-    <parent link="wam/bhand/finger_2/dist_link"/>
-    <child link="wam/bhand/finger_2/tip_link"/>
-    <origin rpy="0 0 0" xyz="0.05 0.0 0.0"/>
-  </joint>
-  <link name="wam/bhand/finger_2/tip_link">
-    <inertial>
-      <mass value="1E-6"/>
-      <inertia ixx="1E-6" ixy="0" ixz="0" iyy="1E-6" iyz="0" izz="1E-6"/>
-    </inertial>
-  </link>
-  <joint name="wam/bhand/finger_3/med_joint" type="revolute">
-    <parent link="wam/bhand/bhand_palm_link"/>
-    <child link="wam/bhand/finger_3/med_link"/>
-    <origin rpy="1.57079632679 0 1.57079632679" xyz="0 0.05 0.0754"/>
-    <axis xyz="0 0 1"/>
-    <limit effort="5" lower="0" upper="2.44346095279" velocity="5.00"/>
-    <dynamics damping="0.11" friction="0"/>
-  </joint>
-  <gazebo reference="wam/bhand/finger_3/med_joint">
-    <provideFeedback>true</provideFeedback>
-    <implicitSpringDamper>true</implicitSpringDamper>
-    <!--<kp>0.0</kp>[> CFM <]-->
-    <!--<kd>0.0</kd>[> ERP <]-->
-    <!--<cfmDamping>true</cfmDamping>-->
-    <!--<dynamics damping="5.5" friction="1"/>-->
-  </gazebo>
-  <gazebo reference="wam/bhand/finger_3/med_link">
-    <mu1>0.8</mu1>
-    <mu2>0.8</mu2>
-  </gazebo>
-  <link name="wam/bhand/finger_3/med_link">
-    <inertial>
-      <origin xyz="0.023133 0.00078642 0.00052792"/>
-      <mass value="0.062139"/>
-      <inertia ixx="4.872e-006" ixy="1.7103e-006" ixz="3.4041e-008" iyy="7.6588e-005" iyz="2.3133e-008" izz="7.7733e-005"/>
-    </inertial>
-    <visual>
-      <material name="WAMGrey">
-        <color rgba="0.9 0.9 0.9 0.0"/>
-      </material>
-      <geometry>
-        <mesh filename="package://barrett_model/models/sw_meshes/bhand/bhand_finger_med_link_fine.stl"/>
-      </geometry>
-    </visual>
-    <collision>
-      <geometry>
-        <mesh filename="package://barrett_model/models/sw_meshes/bhand/bhand_finger_med_link_convex.dae"/>
-      </geometry>
-    </collision>
-  </link>
-  <joint name="wam/bhand/finger_3/dist_joint" type="revolute">
-    <parent link="wam/bhand/finger_3/med_link"/>
-    <child link="wam/bhand/finger_3/dist_link"/>
-    <origin rpy="0 0 0.785398163397" xyz="0.06994 0.003 0.0"/>
-    <axis xyz="0 0 1"/>
-    <limit effort="5" lower="0" upper="0.837758040957" velocity="5.00"/>
-    <dynamics damping="0.11" friction="0"/>
-  </joint>
-  <gazebo reference="wam/bhand/finger_3/dist_joint">
-    <provideFeedback>true</provideFeedback>
-    <implicitSpringDamper>true</implicitSpringDamper>
-    <!--<kp>0.0</kp>[> CFM <]-->
-    <!--<kd>0.0</kd>[> ERP <]-->
-    <!--<cfmDamping>true</cfmDamping>-->
-    <!--<dynamics damping="5.5" friction="1"/>-->
-  </gazebo>
-  <gazebo reference="wam/bhand/finger_3/dist_link">
-    <mu1>0.8</mu1>
-    <mu2>0.8</mu2>
-    <selfCollide>true</selfCollide>
-  </gazebo>
-  <link name="wam/bhand/finger_3/dist_link">
-    <inertial>
-      <origin rpy="0 0 0" xyz="0.022825 0.0010491 0.0004203"/>
-      <mass value="0.041377"/>
-      <inertia ixx="3.1582e-006" ixy="1.4308e-006" ixz="1.0106e-007" iyy="3.8376e-005" iyz="0" izz="3.7275e-005"/>
-    </inertial>
-    <visual>
-      <origin rpy="0 0 -0.785398163397"/>
-      <material name="WAMGrey">
-        <color rgba="0.9 0.9 0.9 0.0"/>
-      </material>
-      <geometry>
-        <mesh filename="package://barrett_model/models/sw_meshes/bhand/bhand_finger_dist_link_fine.stl"/>
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