Commit message: 差速底盘+机械臂+末端相机

File: barrett_model/robots/mobile_7dof_wam_kinectv1.urdf.xacro (robot description, xacro)
@@ -14,5 +14,5 @@
     <parent link="base_footprint"/>
     <child link="wam/base_link"/>
-    <origin rpy="0 0 0" xyz="0.0 0.0 0.103"/>
+    <origin rpy="0 0 0" xyz="0.0 0.0 0.03"/>
   </joint>
   <gazebo reference="wam/wam_fixed_joint">
@@ -23,5 +23,5 @@
     <inertial>
       <origin xyz="0 0 0"/>
-      <mass value="1"/>
+      <mass value="10"/>
       <inertia ixx="0.1" ixy="0" ixz="0" iyy="0.1" iyz="0" izz="0.1"/>
     </inertial>

File: barrett_model/robots/mobile_chassis.urdf.xacro (robot description, xacro)
@@ -227,9 +227,9 @@
         </gazebo>
         <!-- Wheel Definitions -->
-        <wheel lr="right"  translateY="-1" />
-        <wheel lr="left"  translateY="1" />
+        <wheel lr="right"  translateY="-4" />
+        <wheel lr="left"  translateY="4" />
         <!-- Casters Definitions -->
-        <caster fb="front"  translateX="-1" />
-        <caster fb="back"  translateX="1" />
+        <caster fb="front"  translateX="-4" />
+        <caster fb="back"  translateX="4" />
         <!--  plates and standoff Definitions -->
         <!-- <mrobot_standoff_2in parent="base_link" number="1" x_loc="-${standoff_x/2 + 0.03}" y_loc="-${standoff_y - 0.03}" z_loc="${plate_height/2}"/>
