Commit message: 移动底盘+arm

File: barrett_model/models/kinect.urdf.xacro (robot description, xacro)
@@ -43,5 +43,5 @@
   </xacro:macro>
   <!-- [2]  pose from camera to robot -->
-  <xacro:property name="cam_px" value="0" />
+  <xacro:property name="cam_px" value="0.02" />
 	<xacro:property name="cam_pz" value="0" />
 	<xacro:property name="cam_or" value="0" />
@@ -50,7 +50,7 @@
   <xacro:property name="kinect_cam_py" value="-0.0125"/>
   <!-- [3]  Parameterised in part by the values in turtlebot_properties.urdf.xacro -->
-  <xacro:macro name="sensor_kinect" params="parent cam_pz_input">
+  <xacro:macro name="sensor_kinect" params="parent cam_px_input cam_pz_input">
     <joint name="camera_rgb_joint" type="fixed">
-      <origin xyz="${cam_px} ${kinect_cam_py} ${cam_pz_input}" rpy="${cam_or} ${cam_op} ${cam_oy}"/>
+      <origin xyz="${cam_px_input} ${kinect_cam_py} ${cam_pz_input}" rpy="${cam_or} ${cam_op} ${cam_oy}"/>
       <parent link="${parent}"/>
       <child link="camera_rgb_frame" />

File: barrett_model/robots/mobile_7dof_wam_kinectv1.urdf.xacro (robot description, xacro)
@@ -8,15 +8,16 @@
     <color rgba="0.7 0.7 0.7 1.0"/>
   </material>
-  <!-- Root link is in the world frame-->
-  <!-- <link name="world"/>
+  <!-- <xacro:include filename="$(find barrett_model)/robots/test_robot.urdf.xacro" /> -->
+	<xacro:include filename="$(find barrett_model)/robots/mobile_chassis.urdf.xacro" />
+  <mrobot_body/>
   <joint name="wam/wam_fixed_joint" type="fixed">
-    <parent link="world"/>
+    <parent link="base_footprint"/>
     <child link="wam/base_link"/>
-    <origin rpy="0 0 0" xyz="0.0 0.0 0"/>
+    <origin rpy="0 0 0" xyz="0.0 0.0 0.103"/>
   </joint>
   <gazebo reference="wam/wam_fixed_joint">
     <provideFeedback>true</provideFeedback>
     <implicitSpringDamper>true</implicitSpringDamper>
-  </gazebo> -->
+  </gazebo>
   <link name="wam/base_link">
     <inertial>
@@ -35,5 +36,5 @@
     <collision>
       <geometry>
-        <mesh filename="package://barrett_model/models/sw_meshes/base_link_convex.dae"/>
+        <!-- <mesh filename="package://barrett_model/models/sw_meshes/base_link_convex.dae"/> -->
       </geometry>
     </collision>

Commit message: 添加单个床world

File: barrett_model/models/kinect.urdf.xacro (robot description, xacro)
@@ -75,5 +75,5 @@
         </geometry>
       </visual>
-  	  <collision>
+  	  <collision>s
         <origin xyz="0.0 0.0 0.0" rpy="0 0 0"/>
   	    <geometry>

File: barrett_model/robots/mobile_7dof_wam_kinectv1.urdf.xacro (robot description, xacro)
@@ -117,5 +117,7 @@
     <origin rpy="1.57079632679 0 0" xyz="0 0 0"/>
     <axis xyz="0 0 1"/>
-    <limit effort="45" lower="-2.79999681239" upper="2.79999681239" velocity="2.0"/>
+    <!-- <limit effort="45" lower="-2.79999681239" upper="2.79999681239" velocity="2.0"/> -->
+    <limit effort="45" lower="-3.9999681239" upper="3.79999681239" velocity="2.0"/>
+    <!-- this is joint 3 -->
     <dynamics damping="1.65" friction="0"/>
   </joint>
@@ -204,5 +206,7 @@
     <origin rpy="1.57079632679 0 0" xyz="-0.045 -0.3 0"/>
     <axis xyz="0 0 1"/>
-    <limit effort="10" lower="-4.55000354678" upper="1.25000481028" velocity="2.0"/>
+    <!-- <limit effort="10" lower="-4.55000354678" upper="1.25000481028" velocity="2.0"/> -->
+    <limit effort="10" lower="-4.55000354678" upper="2.25000481028" velocity="2.0"/>
+    <!-- this is joint 5 -->
     <dynamics damping="0.55" friction="0"/>
   </joint>
